File: Hardware/KiCad/v0.3/Cryologger AWS.kicad_pcb (KiCad board)
At the start: 2 copper layers, 133.3 x 79.4 mm, 23 parts, among them J1 Screw_Terminal_01x10, J2 Screw_Terminal_01x10, J3 Screw_Terminal_01x02, J4 Conn_01x20, U1 Adafruit_Feather_Header, U2 Adafruit_Feather_Header, U3 RockBLOCK_Footprint, U4 ROCKBLOCK_9603, U5 Adafruit_DPS310, U6 Pololu_D36V6x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

Commit message: Minor updates to KiCad files
Changed text on silkscreen and removed ground from hole pads.
Parts:
- removed the REF** at (102.9, 115.6)
Connections:
- H1 pad 1: GND -> unconnected-(H1-Pad1)
- H2 pad 1: GND -> unconnected-(H2-Pad1)
- H3 pad 1: GND -> unconnected-(H3-Pad1)
- H4 pad 1: GND -> unconnected-(H4-Pad1)
Other:
- board text added: "Contact if found: Adam Garbo Ottawa, Ontario, Canada adam@cryologger.org"
- board text removed: "Contact if found: Adam Garbo Carleton University Ottawa, Ontario, Canada adam.garbo@carleton.ca"
