File: Hardware/KiCad/v0.3/_autosave-Cryologger AWS.kicad_sch (KiCad schematic)
At the start: 20 parts, among them J1 Screw_Terminal_01x10, J2 Screw_Terminal_01x10, J3 Screw_Terminal_01x02, J4 Conn_01x20, U1 Adafruit_Feather_Header, U2 Adafruit_Feather_Header, U3 RockBLOCK_Footprint, U4 ROCKBLOCK_9603, U5 Adafruit_DPS310, U6 Pololu_D36V6x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

Commit message: Minor updates to KiCad files
Changed text on silkscreen and removed ground from hole pads.
Connections:
- net GND: now also H1.1, H2.1, H3.1, H4.1
Changed lines of the file:
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@@
 (kicad_sch (version 20211123) (generator eeschema)
   (paper "A4")
+  (junction (at 276.86 93.98) (diameter 0) (color 0 0 0 0)
+  )
   (junction (at 127 171.45) (diameter 0) (color 0 0 0 0)
   )
@@
   (junction (at 30.48 189.23) (diameter 0) (color 0 0 0 0)
   )
+  (junction (at 276.86 88.9) (diameter 0) (color 0 0 0 0)
+  )
+  (junction (at 276.86 83.82) (diameter 0) (color 0 0 0 0)
+  )
   (junction (at 40.64 142.24) (diameter 0) (color 0 0 0 0)
   )
@@
     (stroke (width 0) (type default) (color 0 0 0 0))
   )
+  (wire (pts (xy 276.86 83.82) (xy 276.86 88.9))
+    (stroke (width 0) (type default) (color 0 0 0 0))
+  )
   (wire (pts (xy 72.39 166.37) (xy 72.39 176.53))
     (stroke (width 0) (type default) (color 0 0 0 0))
@@
     (stroke (width 0) (type default) (color 0 0 0 0))
   )
+  (wire (pts (xy 276.86 93.98) (xy 276.86 96.52))
+    (stroke (width 0) (type default) (color 0 0 0 0))
+  )
   (wire (pts (xy 41.91 132.08) (xy 39.37 132.08))
     (stroke (width 0) (type default) (color 0 0 0 0))
@@
     (stroke (width 0) (type default) (color 0 0 0 0))
   )
+  (wire (pts (xy 276.86 78.74) (xy 276.86 83.82))
+    (stroke (width 0) (type default) (color 0 0 0 0))
+  )
   (wire (pts (xy 29.21 57.15) (xy 26.67 57.15))
     (stroke (width 0) (type default) (color 0 0 0 0))
@@
   )
   (wire (pts (xy 73.66 119.38) (xy 71.12 119.38))
+    (stroke (width 0) (type default) (color 0 0 0 0))
+  )
+  (wire (pts (xy 276.86 88.9) (xy 276.86 93.98))
     (stroke (width 0) (type default) (color 0 0 0 0))
   )
@@
     (pin "1")
   )
+  (symbol (lib_id "power:GND") (at 276.86 96.52 0) (unit 1)
+    (in_bom yes) (on_board yes)
+    (property "Reference" "#PWR036" (id 0) (at 276.86 102.87 0)
+      (effects (font (size 1.27 1.27)) hide)
+    )
+    (property "Value" "GND" (id 1) (at 276.987 100.9142 0))
+    (property "Footprint" "" (id 2) (at 276.86 96.52 0)
+      (effects (font (size 1.27 1.27)) hide)
+    )
+    (property "Datasheet" "" (id 3) (at 276.86 96.52 0)
+      (effects (font (size 1.27 1.27)) hide)
+    )
+    (pin "1")
+  )
   (symbol (lib_id "Connector:Screw_Terminal_01x02") (at 114.935 118.11 0) (mirror y) (unit 1)
     (in_bom yes) (on_board yes) (fields_autoplaced)
@@
       (reference "#PWR035") (unit 1) (value "+BATT") (footprint "")
     )
+    (path "/00000000-0000-0000-0000-0000607d7b69"
+      (reference "#PWR036") (unit 1) (value "GND") (footprint "")
+    )
     (path "/00000000-0000-0000-0000-00006081e600"
